File: pogoprog.kicad_sch (KiCad schematic)
At the start: 10 parts, among them J3 Conn_02x06_Odd_Even, M1 Arduino_Mini

Commit message: Converted back to 2 layer, as I got the connector size wrong.
Should be 2x6 x 2.54mm pitch
Parts:
- added H1, H2: MountingHole, MountingHole:MountingHole_2.2mm_M2, symbol Mechanical:MountingHole
- J3: footprint Connector_PinHeader_1.27mm:PinHeader_2x06_P1.27mm_Vertical -> Connector_PinHeader_2.54mm:PinHeader_2x06_P2.54mm_Vertical
- PRG1: renamed from JP4; value Jumper_2_Open -> PRG
- R1, R2, R3: footprint Resistor_SMD:R_0603_1608Metric -> Resistor_SMD:R_0805_2012Metric_Pad1.20x1.40mm_HandSolder
Changed lines of the file:
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@@
   (paper "A4")
   (title_block
-    (date "sam. 04 avril 2015")
+    (date "2023-05-11")
+    (rev "v1.3a")
   )
   (no_connect (at 122.555 87.63))
@@
       (effects (font (size 1.27 1.27)))
     )
-    (property "Footprint" "Connector_PinHeader_1.27mm:PinHeader_2x06_P1.27mm_Vertical" (at 133.985 55.88 0)
+    (property "Footprint" "Connector_PinHeader_2.54mm:PinHeader_2x06_P2.54mm_Vertical" (at 133.985 55.88 0)
       (effects (font (size 1.27 1.27)) hide)
     )
@@
     )
   )
+  (symbol (lib_id "Mechanical:MountingHole") (at 74.93 50.8 0) (unit 1)
+    (in_bom yes) (on_board yes) (dnp no) (fields_autoplaced)
+    (property "Reference" "H1" (at 77.47 50.1563 0)
+      (effects (font (size 1.27 1.27)) (justify left))
+    )
+    (property "Value" "MountingHole" (at 77.47 52.0773 0)
+      (effects (font (size 1.27 1.27)) (justify left))
+    )
+    (property "Footprint" "MountingHole:MountingHole_2.2mm_M2" (at 74.93 50.8 0)
+      (effects (font (size 1.27 1.27)) hide)
+    )
+    (property "Datasheet" "~" (at 74.93 50.8 0)
+      (effects (font (size 1.27 1.27)) hide)
+    )
+    (instances
+      (project "pogoprog"
+        (path "/0d35483a-0b12-46cc-b9f2-896fd6831779"
+          (reference "H1") (unit 1)
+        )
+      )
+    )
+  )
   (symbol (lib_id "Device:R") (at 201.295 93.98 0) (mirror y) (unit 1)
     (in_bom yes) (on_board yes) (dnp no) (fields_autoplaced)
@@
       (effects (font (size 1.27 1.27)) (justify left))
     )
-    (property "Footprint" "Resistor_SMD:R_0603_1608Metric" (at 203.073 93.98 90)
+    (property "Footprint" "Resistor_SMD:R_0805_2012Metric_Pad1.20x1.40mm_HandSolder" (at 203.073 93.98 90)
       (effects (font (size 1.27 1.27)) hide)
     )
@@
       (effects (font (size 1.27 1.27)) (justify left))
     )
-    (property "Footprint" "Resistor_SMD:R_0603_1608Metric" (at 212.598 93.98 90)
+    (property "Footprint" "Resistor_SMD:R_0805_2012Metric_Pad1.20x1.40mm_HandSolder" (at 212.598 93.98 90)
       (effects (font (size 1.27 1.27)) hide)
     )
@@
   (symbol (lib_id "Jumper:Jumper_2_Open") (at 91.44 115.57 0) (unit 1)
     (in_bom yes) (on_board yes) (dnp no) (fields_autoplaced)
-    (property "Reference" "JP4" (at 91.44 110.2192 0)
-      (effects (font (size 1.27 1.27)))
-    )
-    (property "Value" "Jumper_2_Open" (at 91.44 112.7561 0)
+    (property "Reference" "PRG1" (at 91.44 110.9091 0)
+      (effects (font (size 1.27 1.27)))
+    )
+    (property "Value" "PRG" (at 91.44 112.8301 0)
       (effects (font (size 1.27 1.27)))
     )
@@
       (project "pogoprog"
         (path "/0d35483a-0b12-46cc-b9f2-896fd6831779"
-          (reference "JP4") (unit 1)
+          (reference "PRG1") (unit 1)
         )
       )
@@
       (effects (font (size 1.27 1.27)) (justify left))
     )
-    (property "Footprint" "Resistor_SMD:R_0603_1608Metric" (at 222.123 93.98 90)
+    (property "Footprint" "Resistor_SMD:R_0805_2012Metric_Pad1.20x1.40mm_HandSolder" (at 222.123 93.98 90)
       (effects (font (size 1.27 1.27)) hide)
     )
@@
         )
       )
+    )
+  )
+  (symbol (lib_id "Mechanical:MountingHole") (at 74.93 59.055 0) (unit 1)
+    (in_bom yes) (on_board yes) (dnp no) (fields_autoplaced)
+    (property "Reference" "H2" (at 77.47 58.4113 0)
+      (effects (font (size 1.27 1.27)) (justify left))
+    )
+    (property "Value" "MountingHole" (at 77.47 60.3323 0)
+      (effects (font (size 1.27 1.27)) (justify left))
+    )
+    (property "Footprint" "MountingHole:MountingHole_2.2mm_M2" (at 74.93 59.055 0)
+      (effects (font (size 1.27 1.27)) hide)
+    )
+    (property "Datasheet" "~" (at 74.93 59.055 0)
+      (effects (font (size 1.27 1.27)) hide)
+    )
+    (instances
+      (project "pogoprog"
+        (path "/0d35483a-0b12-46cc-b9f2-896fd6831779"
+          (reference "H2") (unit 1)
+        )
+      )

Commit message: Added pads for a common-anode 8mm RGB LED
Parts:
- added D4: LED_RAGB, aalib:LED_D8.0mm-4_RGB, symbol Device:LED_RAGB
Connections:
- net +5V: now also D4.2 (A)
- net at D3.2 (A), R3.2: now also D4.4 (BK)
- net at D2.2 (A), R2.2: now also D4.1 (RK)
- net at D1.2 (A), R1.2: now also D4.3 (GK)
Other:
- moved on the sheet: R1, R2
Changed lines of the file:
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@@
     (rev "v1.3a")
+  )
+  (junction (at 201.295 100.33) (diameter 0) (color 0 0 0 0)
+  )
+  (junction (at 210.82 96.52) (diameter 0) (color 0 0 0 0)
+  )
+  (junction (at 220.345 93.345) (diameter 0) (color 0 0 0 0)
   )
   (no_connect (at 122.555 87.63))
@@
     (stroke (width 0) (type default))
   )
+  (wire (pts (xy 248.92 100.33) (xy 248.92 79.375))
+    (stroke (width 0) (type default))
+  )
   (wire (pts (xy 196.215 80.645) (xy 220.345 80.645))
     (stroke (width 0) (type default))
@@
     (stroke (width 0) (type default))
   )
-  (wire (pts (xy 201.295 97.79) (xy 201.295 102.235))
-    (stroke (width 0) (type default))
-  )
-  (wire (pts (xy 210.82 97.79) (xy 210.82 102.235))
+  (wire (pts (xy 201.295 97.79) (xy 201.295 100.33))
+    (stroke (width 0) (type default))
+  )
+  (wire (pts (xy 210.82 93.345) (xy 210.82 96.52))
     (stroke (width 0) (type default))
   )
@@
     (stroke (width 0) (type default))
   )
+  (wire (pts (xy 243.84 65.405) (xy 243.84 69.215))
+    (stroke (width 0) (type default))
+  )
   (wire (pts (xy 104.775 95.25) (xy 122.555 95.25))
     (stroke (width 0) (type default))
@@
   )
   (wire (pts (xy 117.475 113.03) (xy 122.555 113.03))
+    (stroke (width 0) (type default))
+  )
+  (wire (pts (xy 201.295 100.33) (xy 248.92 100.33))
     (stroke (width 0) (type default))
   )
@@
     (stroke (width 0) (type solid))
   )
+  (wire (pts (xy 201.295 100.33) (xy 201.295 102.235))
+    (stroke (width 0) (type default))
+  )
+  (wire (pts (xy 210.82 96.52) (xy 210.82 102.235))
+    (stroke (width 0) (type default))
+  )
   (wire (pts (xy 104.775 100.33) (xy 122.555 100.33))
     (stroke (width 0) (type default))
@@
     (stroke (width 0) (type default))
   )
-  (wire (pts (xy 210.82 90.17) (xy 210.82 83.185))
+  (wire (pts (xy 210.82 85.725) (xy 210.82 83.185))
     (stroke (width 0) (type default))
   )
@@
     (stroke (width 0) (type default))
   )
+  (wire (pts (xy 238.76 96.52) (xy 238.76 79.375))
+    (stroke (width 0) (type default))
+  )
+  (wire (pts (xy 220.345 93.345) (xy 220.345 102.235))
+    (stroke (width 0) (type default))
+  )
   (wire (pts (xy 147.955 100.33) (xy 160.655 100.33))
     (stroke (width 0) (type default))
   )
-  (wire (pts (xy 220.345 97.79) (xy 220.345 102.235))
+  (wire (pts (xy 220.345 92.075) (xy 220.345 93.345))
     (stroke (width 0) (type default))
   )
   (wire (pts (xy 147.955 90.17) (xy 160.655 90.17))
+    (stroke (width 0) (type default))
+  )
+  (wire (pts (xy 243.84 93.345) (xy 243.84 79.375))
     (stroke (width 0) (type default))
   )
@@
     (stroke (width 0) (type solid))
   )
+  (wire (pts (xy 220.345 93.345) (xy 243.84 93.345))
+    (stroke (width 0) (type default))
+  )
   (wire (pts (xy 83.185 112.395) (xy 83.185 115.57))
     (stroke (width 0) (type default))
   )
-  (wire (pts (xy 220.345 90.17) (xy 220.345 80.645))
+  (wire (pts (xy 210.82 96.52) (xy 238.76 96.52))
+    (stroke (width 0) (type default))
+  )
+  (wire (pts (xy 220.345 84.455) (xy 220.345 80.645))
     (stroke (width 0) (type default))
   )
@@
         (path "/0d35483a-0b12-46cc-b9f2-896fd6831779"
           (reference "J3") (unit 1)
+        )
+      )
+    )
+  )
+  (symbol (lib_id "Device:LED_RAGB") (at 243.84 74.295 90) (unit 1)
+    (in_bom yes) (on_board yes) (dnp no) (fields_autoplaced)
+    (property "Reference" "D4" (at 252.222 73.0829 90)
+      (effects (font (size 1.27 1.27)) (justify right))
+    )
+    (property "Value" "LED_RAGB" (at 252.222 75.5071 90)
+      (effects (font (size 1.27 1.27)) (justify right))
+    )
+    (property "Footprint" "aalib:LED_D8.0mm-4_RGB" (at 245.11 74.295 0)
+      (effects (font (size 1.27 1.27)) hide)
+    )
+    (property "Datasheet" "~" (at 245.11 74.295 0)
+      (effects (font (size 1.27 1.27)) hide)
+    )
+    (pin "1")
+    (pin "2")
+    (pin "3")
+    (pin "4")
+    (instances
+      (project "pogoprog"
+        (path "/0d35483a-0b12-46cc-b9f2-896fd6831779"
+          (reference "D4") (unit 1)
         )
       )
@@
     )
   )
-  (symbol (lib_id "Device:R") (at 210.82 93.98 0) (mirror y) (unit 1)
-    (in_bom yes) (on_board yes) (dnp no) (fields_autoplaced)
-    (property "Reference" "R2" (at 209.042 93.1453 0)
-      (effects (font (size 1.27 1.27)) (justify left))
-    )
-    (property "Value" "R" (at 209.042 95.6822 0)
-      (effects (font (size 1.27 1.27)) (justify left))
-    )
-    (property "Footprint" "Resistor_SMD:R_0805_2012Metric_Pad1.20x1.40mm_HandSolder" (at 212.598 93.98 90)
-      (effects (font (size 1.27 1.27)) hide)
-    )
-    (property "Datasheet" "~" (at 210.82 93.98 0)
+  (symbol (lib_id "Device:R") (at 210.82 89.535 0) (unit 1)
+    (in_bom yes) (on_board yes) (dnp no)
+    (property "Reference" "R2" (at 212.598 88.7003 0)
+      (effects (font (size 1.27 1.27)) (justify left))
+    )
+    (property "Value" "R" (at 212.598 91.2372 0)
+      (effects (font (size 1.27 1.27)) (justify left))
+    )
+    (property "Footprint" "Resistor_SMD:R_0805_2012Metric_Pad1.20x1.40mm_HandSolder" (at 209.042 89.535 90)
+      (effects (font (size 1.27 1.27)) hide)
+    )
+    (property "Datasheet" "~" (at 210.82 89.535 0)
       (effects (font (size 1.27 1.27)) hide)
     )
@@
     )
   )
-  (symbol (lib_id "Device:R") (at 220.345 93.98 0) (mirror y) (unit 1)
+  (symbol (lib_id "power:+5V") (at 243.84 65.405 0) (unit 1)
+    (in_bom yes) (on_board yes) (dnp no)
+    (property "Reference" "#PWR07" (at 243.84 69.215 0)
+      (effects (font (size 1.27 1.27)) hide)
+    )
+    (property "Value" "+5V" (at 243.84 61.849 90)
+      (effects (font (size 1.27 1.27)) (justify left))
+    )
+    (property "Footprint" "" (at 243.84 65.405 0)
+      (effects (font (size 1.27 1.27)) hide)
+    )
+    (property "Datasheet" "" (at 243.84 65.405 0)
+      (effects (font (size 1.27 1.27)) hide)
+    )
+    (pin "1")
+    (instances
+      (project "pogoprog"
+        (path "/0d35483a-0b12-46cc-b9f2-896fd6831779"
+          (reference "#PWR07") (unit 1)
+        )
+      )
+    )
+  )
+  (symbol (lib_id "Device:R") (at 220.345 88.265 0) (mirror y) (unit 1)
     (in_bom yes) (on_board yes) (dnp no) (fields_autoplaced)
-    (property "Reference" "R1" (at 218.567 93.1453 0)
-      (effects (font (size 1.27 1.27)) (justify left))
-    )
-    (property "Value" "R" (at 218.567 95.6822 0)
-      (effects (font (size 1.27 1.27)) (justify left))
-    )
-    (property "Footprint" "Resistor_SMD:R_0805_2012Metric_Pad1.20x1.40mm_HandSolder" (at 222.123 93.98 90)
-      (effects (font (size 1.27 1.27)) hide)
-    )
-    (property "Datasheet" "~" (at 220.345 93.98 0)
-      (effects (font (size 1.27 1.27)) hide)
-    )
+    (property "Reference" "R1" (at 218.567 87.4303 0)
+      (effects (font (size 1.27 1.27)) (justify left))
+    )
+    (property "Value" "R" (at 218.567 89.9672 0)
+      (effects (font (size 1.27 1.27)) (justify left))
+    )
+    (property "Footprint" "Resistor_SMD:R_0805_2012Metric_Pad1.20x1.40mm_HandSolder" (at 222.123 88.265 90)
+      (effects (font (size 1.27 1.27)) hide)
+    )
+    (property "Datasheet" "~" (at 220.345 88.265 0)
+      (effects (font (size 1.27 1.27)) hide)
+    )

Commit message: Last minute tweaks
Improved silkscreen for LED labels.
Added text to back showing connector pinout
Moved M1
Renamed J3 to J1
Parts:
- renumbered J3 to J1
Changed lines of the file:
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@@
   (symbol (lib_id "Connector_Generic:Conn_02x06_Odd_Even") (at 133.985 55.88 0) (unit 1)
     (in_bom yes) (on_board yes) (dnp no)
-    (property "Reference" "J3" (at 135.255 66.675 0)
+    (property "Reference" "J1" (at 135.255 66.675 0)
       (effects (font (size 1.27 1.27)))
     )
@@
       (project "pogoprog"
         (path "/0d35483a-0b12-46cc-b9f2-896fd6831779"
-          (reference "J3") (unit 1)
+          (reference "J1") (unit 1)
         )
       )
